Commit message: feat(kinematics): add closed-form arm kinematics and widen shoulder/elbow to ±135°
With ±90° limits no table position is reachable. The Python package is
installed with ament_cmake_python and the whole test directory now runs.

File: src/lab_simulation/urdf/simple_arm.urdf (robot description, URDF)
Before this commit: robot simple_arm, 6 links, 5 joints
Joints:
- joint joint_2: limit lower=-1.5708 upper=1.5708 effort=15 velocity=2.0 -> lower=-2.356 upper=2.356 effort=15 velocity=2.0
- joint joint_3: limit lower=-1.5708 upper=1.5708 effort=10 velocity=2.0 -> lower=-2.356 upper=2.356 effort=10 velocity=2.0
